File: ControllerPCB.sch (KiCad schematic (older format))
At the start: 23 parts

Commit message: Layout of PCB
Parts:
- D1, D2, D3: renamed from D?; footprint (none) -> Diode_THT:D_5KP_P12.70mm_Horizontal
- J1, J3, J4, J6: renamed from J?; footprint (none) -> Connector_PinHeader_2.54mm:PinHeader_1x02_P2.54mm_Vertical
- J10: renamed from J?; footprint (none) -> Connector_PinHeader_2.54mm:PinHeader_1x06_P2.54mm_Vertical
- J2, J8, J9: renamed from J?; footprint (none) -> Connector_PinHeader_2.54mm:PinHeader_1x04_P2.54mm_Vertical
- J5: renamed from J?; footprint (none) -> Connector_PinHeader_2.54mm:PinHeader_1x03_P2.54mm_Vertical
- J7: renamed from J?; footprint ASSMANN_A-2004-2-4-LPS-N-R -> A-2004-2-4-LPS-N-R:ASSMANN_A-2004-2-4-LPS-N-R
- P1: renamed from P?; footprint OST_USB-A1HSW6 -> USB-A1HSW6:OST_USB-A1HSW6
- Q1, Q2: renamed from Q?; footprint Package_TO_SOT_SMD:SOT-23 -> Connector_PinHeader_2.54mm:PinHeader_1x03_P2.54mm_Vertical
- R1, R2, R3, R4: renamed from R?; footprint (none) -> Resistor_THT:R_Axial_DIN0207_L6.3mm_D2.5mm_P10.16mm_Horizontal
- U1: renamed from U?; footprint CONV_BOB-12009 -> BOB-12009:CONV_BOB-12009
- XA1: renamed from XA?; footprint (none) -> Arduino:Arduino_Mega2560_Shield
- XA2: renamed from XA?; footprint (none) -> Arduino:Arduino_Nano_Socket
Connections:
- net ScaleCLK1: now also XA1.D12; no longer XA1.D24
- net ScaleCLK2: now also XA1.D13; no longer XA1.D25
- net ScaleD1: now also XA1.D10; no longer XA1.D22
- net ScaleD2: now also XA1.D11; no longer XA1.D23

Commit message: V2
Parts:
- removed D1, D2, D3: DIODE, Diode_THT:D_5KP_P12.70mm_Horizontal, symbol pspice:DIODE
- removed J4: Conn_01x02_Male, Connector_PinHeader_2.54mm:PinHeader_1x02_P2.54mm_Vertical, symbol Connector:Conn_01x02_Male
- added D1, D2, D3, D4: D, Diode_THT:D_DO-15_P15.24mm_Horizontal, symbol Device:D
- added J11, J12: Conn_01x02_Male, Connector_PinHeader_2.54mm:PinHeader_1x02_P2.54mm_Vertical, symbol Connector:Conn_01x02_Male
- added J4: Conn_01x03_Male, Connector_PinHeader_2.54mm:PinHeader_1x03_P2.54mm_Vertical, symbol Connector:Conn_01x03_Male
Connections:
- net TX0 is gone; now on net TX1: XA2.D1 (D1_TX0)
- net +3V3: no longer J2.1 (Pin_1), J5.1 (Pin_1), R1.1, R2.1, XA2.3V3 (3.3V)
- net +5V: now also J2.4 (Pin_4), J5.3 (Pin_3), J6.2 (Pin_2), R1.1, R2.1, D3.1 (K), D4.1 (K), J11.2 (Pin_2), J12.2 (Pin_2), J4.2 (Pin_2); no longer J6.1 (Pin_1), XA1.5V1 (5V), XA1.5V3 (5V), XA1.5V4 (5V), XA2.5V
- net DialCLK: now also U1.HV1; no longer U1.HV2
- net DialData: now also U1.HV2; no longer U1.HV1
- net Fans-: now also J6.1 (Pin_1), D1.2 (A), D4.2 (A), J11.1 (Pin_1), J12.1 (Pin_1); no longer J6.2 (Pin_2)
- net GND: now also J1.1 (Pin_1), J2.1 (Pin_1), J3.1 (Pin_1), J5.1 (Pin_1), J4.1 (Pin_1); no longer J1.2 (Pin_2), J2.2 (Pin_2), J3.2 (Pin_2), J5.3 (Pin_3)
- net RollerMotor-: now also D2.2 (A), D3.2 (A)
- net ScaleCLK1: now also XA2.D4; no longer XA1.D12
- net ScaleCLK2: now also XA2.D7; no longer XA1.D13
- net ScaleD1: now also XA2.D6; no longer XA1.D10
- net ScaleD2: now also XA2.D5; no longer XA1.D11
- net ScrewMotor: now also J1.2 (Pin_2); no longer J1.1 (Pin_1)
- net SlackS0: now also J2.2 (Pin_2); no longer J2.3 (Pin_3)
- net SlackS1: now also J2.3 (Pin_3); no longer J2.4 (Pin_4)
- net SpollerMotor: now also J3.2 (Pin_2); no longer J3.1 (Pin_1)
- net Vin: now also XA2.VIN, J4.3 (Pin_3)
- net at U1.LV1: now also P1.2 (D-); no longer P1.3 (D+)
- net LV2: now reaches U1.LV2
- net LV2: now also P1.3 (D+); no longer P1.2 (D-)
- net at Q2.3 (D): now also D2.1 (K)
- net at Q1.3 (D): now also D1.1 (K)

Commit message: Add plot files
Connections:
- net UartToNano: now reaches XA1.D14 (D14_TX3)
- net UartToNano: now also XA2.D0 (D0_RX0)
- net UartToMega: now reaches XA1.D15 (D15_RX3)
- net UartToMega: now also XA2.D1 (D1_TX0)
- net RX1: no longer names the net of XA1.D19 (D19_RX1)
- net RX1: no longer XA2.D0 (D0_RX0)
- net TX1: no longer names the net of XA1.D18 (D18_TX1)
- net TX1: no longer XA2.D1 (D1_TX0)
Changed lines of the file:
@@
 Text GLabel 4150 2950 0    50   Input ~ 0
 TactSignal
-Text GLabel 4150 1850 0    50   Input ~ 0
-RX1
-Text GLabel 4150 1950 0    50   Input ~ 0
-TX1
+Text GLabel 4150 2250 0    50   Input ~ 0
+UartToMega
+Text GLabel 4150 2350 0    50   Input ~ 0
+UartToNano
 Text GLabel 16950 2600 0    50   Input ~ 0
-RX1
+UartToNano
 Text GLabel 16950 2700 0    50   Input ~ 0
-TX1
+UartToMega
 Text Notes 19450 10200 2    197  ~ 0
 Roller Motor Output

Commit message: Fixed two unconnected pads
Connections:
- net RollerMotor is gone; now on net RollerSpeed: Q2.1 (G), R4.1
- net FansSpeed: now also XA1.D6
- net SlackS0: now also XA1.A1
- net SlackS1: now also XA1.A2
- net RollerSpeed: now reaches XA1.D7
Changed lines of the file:
@@
 	18700 8600 18950 8600
 Text GLabel 18400 8600 0    50   Input ~ 0
-RollerMotor
+RollerSpeed
 Wire Wire Line
 	18400 8600 18700 8600
@@
 Text GLabel 6750 1650 2    50   Input ~ 0
 EncoderA
+Text GLabel 4150 3050 0    50   Input ~ 0
+SlackS0
+Text GLabel 4150 3150 0    50   Input ~ 0
+SlackS1
+Text GLabel 6750 2050 2    50   Input ~ 0
+FansSpeed
+Text GLabel 6750 2150 2    50   Input ~ 0
+RollerSpeed
 $EndSCHEMATC

Commit message: Updated 5V and 5Vin
Connections:
- net +5V: now also XA1.5V1 (5V); no longer D3.1 (K), D4.1 (K), J11.2 (Pin_2), J12.2 (Pin_2), J4.2 (Pin_2), J6.2 (Pin_2), J7.1
- net Vin: now also J7.8
- new net 5Vin: D3.1 (K), D4.1 (K), J11.2 (Pin_2), J12.2 (Pin_2), J4.2 (Pin_2), J6.2 (Pin_2)
Changed lines of the file:
@@
 $EndDescr
-$Comp
-L Arduino:Arduino_Mega2560_Shield XA1
-U 1 1 605A9FAE
-P 5450 3800
-F 0 "XA1" H 5450 1419 60  0000 C CNN
-F 1 "Arduino_Mega2560_Shield" H 5450 1313 60  0000 C CNN
-F 2 "Arduino:Arduino_Mega2560_Shield" H 6150 6550 60  0001 C CNN
-F 3 "https://store.arduino.cc/arduino-mega-2560-rev3" H 6150 6550 60  0001 C CNN
-	1    5450 3800
-	1    0    0    -1
-$EndComp
 $Comp
 L Arduino:Arduino_Nano_Socket XA2
@@
 Wire Wire Line
 	3850 5050 4150 5050
-Wire Wire Line
-	4150 5450 4150 5350
-Connection ~ 4150 5050
-Connection ~ 4150 5150
-Wire Wire Line
-	4150 5150 4150 5050
-Connection ~ 4150 5250
-Wire Wire Line
-	4150 5250 4150 5150
-Connection ~ 4150 5350
-Wire Wire Line
-	4150 5350 4150 5250
 Text GLabel 4150 5950 0    50   Input ~ 0
 Vin
@@
 	18550 7650 19250 7650
 Connection ~ 19250 7650
-$Comp
-L power:+5V #PWR028
-U 1 1 605D0C1F
-P 19900 6900
-F 0 "#PWR028" H 19900 6750 50  0001 C CNN
-F 1 "+5V" H 19915 7073 50  0000 C CNN
-F 2 "" H 19900 6900 50  0001 C CNN
-F 3 "" H 19900 6900 50  0001 C CNN
-	1    19900 6900
-	1    0    0    -1
-$EndComp
 Text Notes 850  9750 0    197  ~ 0
 Pullup Resistors for I2c
@@
 Wire Wire Line
 	10900 13850 11600 13850
-$Comp
-L power:+5V #PWR016
-U 1 1 6060B4B5
-P 11600 13350
-F 0 "#PWR016" H 11600 13200 50  0001 C CNN
-F 1 "+5V" H 11615 13523 50  0000 C CNN
-F 2 "" H 11600 13350 50  0001 C CNN
-F 3 "" H 11600 13350 50  0001 C CNN
-	1    11600 13350
-	1    0    0    -1
-$EndComp
 Wire Wire Line
 	11600 13550 11600 13500
@@
 	9550 3500 9850 3500
 $Comp
-L power:+5V #PWR010
-U 1 1 60628A57
-P 9600 2600
-F 0 "#PWR010" H 9600 2450 50  0001 C CNN
-F 1 "+5V" H 9615 2773 50  0000 C CNN
-F 2 "" H 9600 2600 50  0001 C CNN
-F 3 "" H 9600 2600 50  0001 C CNN
-	1    9600 2600
-	1    0    0    -1
-$EndComp
-Wire Wire Line
-	9600 2600 9850 2600
-$Comp
 L power:GND #PWR011
 U 1 1 6062ADC7
@@
 	1    0    0    -1
 $EndComp
-$Comp
-L power:+5V #PWR013
-U 1 1 6062F2BE
-P 10400 5850
-F 0 "#PWR013" H 10400 5700 50  0001 C CNN
-F 1 "+5V" H 10415 6023 50  0000 C CNN
-F 2 "" H 10400 5850 50  0001 C CNN
-F 3 "" H 10400 5850 50  0001 C CNN
-	1    10400 5850
-	1    0    0    -1
-$EndComp
-Wire Wire Line
-	10400 5850 10100 5850
 Wire Wire Line
 	10100 5950 10250 5950
@@
 Wire Wire Line
 	10150 13550 10800 13550
-Wire Wire Line
-	19900 6900 19900 7250
 $Comp
 L power:+5V #PWR0102
@@
 Text GLabel 6750 2150 2    50   Input ~ 0
 RollerSpeed
+Text GLabel 9850 3300 0    50   Input ~ 0
+Vin
+$Comp
+L power:+5V #PWR0105
+U 1 1 6063DDF5
+P 3750 5650
+F 0 "#PWR0105" H 3750 5500 50  0001 C CNN
+F 1 "+5V" H 3765 5823 50  0000 C CNN
+F 2 "" H 3750 5650 50  0001 C CNN
+F 3 "" H 3750 5650 50  0001 C CNN
+	1    3750 5650
+	1    0    0    -1
+$EndComp
+Wire Wire Line
+	3750 5650 4150 5650
+Text GLabel 10100 5850 2    50   Input ~ 0
+5Vin
+Text GLabel 11600 13350 0    50   Input ~ 0
+5Vin
+Text GLabel 19900 6850 0    50   Input ~ 0
+5Vin
+Wire Wire Line
+	19900 6850 19900 7250
+Wire Wire Line
+	4150 5450 4150 5350
+Connection ~ 4150 5350
+Wire Wire Line
+	4150 5350 4150 5250
+Connection ~ 4150 5250
+Wire Wire Line
+	4150 5250 4150 5150
+Wire Wire Line
+	4150 5150 4150 5050
+Connection ~ 4150 5150
+Connection ~ 4150 5050
+$Comp
+L Arduino:Arduino_Mega2560_Shield XA1
+U 1 1 605A9FAE
+P 5450 3800
+F 0 "XA1" H 5450 1419 60  0000 C CNN
+F 1 "Arduino_Mega2560_Shield" H 5450 1313 60  0000 C CNN
+F 2 "Arduino:Arduino_Mega2560_Shield" H 6150 6550 60  0001 C CNN
+F 3 "https://store.arduino.cc/arduino-mega-2560-rev3" H 6150 6550 60  0001 C CNN
+	1    5450 3800
+	1    0    0    -1
+$EndComp
 $EndSCHEMATC
